Commit message: Post SAR changes (hopefully nothing is broken)

File: src/beep_autonomy/src/description/rover_description.urdf (robot description, URDF)
Before this commit: robot rover, 8 links, 7 joints
Joints:
- joint imu_joint: origin xyz=0.37 0 0.12 -> xyz=0 0 0.12
- joint lidar_joint: origin xyz=0.37 0 0.2 rpy=0 0 0 -> xyz=0 0 0.2 rpy=0 0 0
- joint sensor_joint: origin xyz=0.37 0 0.12 -> xyz=0 0 0.12
